File: main_relay_board.kicad_sch (KiCad schematic)
At the start: 19 parts, among them J101 Screw_Terminal_01x03, J102 Conn_01x04_Socket, J103 Conn_01x04_Socket, J104 Conn_01x08_Socket, J105 Conn_01x04_Socket, J106 Conn_01x04_Socket, J107 Conn_01x06_Socket, J108 Conn_01x04_Socket, J109 Conn_01x04_Socket, J110 Conn_01x04_Socket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

Commit message: finished...
Other:
- moved on the sheet: J105, J107, J109, J110
