File: mcu.kicad_sch (KiCad schematic)
At the start: 17 parts, among them SW301 RST_SW, U301 STM32F205RBTx, U302 MCP9700x-ETT, Y301 8MHz

Commit message: finished...
Parts:
- Y301: LCSC (none) -> C2682775
Changed lines of the file:
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@@
 	(title_block
 		(title "Relay Control Board")
-		(date "2024-07-01")
-		(rev "PA")
+		(date "2024-07-09")
+		(rev "R1")
 		(company "UBC ThunderBikes")
 		(comment 1 "Peter Woolsey")
@@
 			)
 		)
-		(property "LCSC" ""
+		(property "LCSC" "C2682775"
 			(at 43.18 77.47 90)
 			(effects
