File: power.kicad_sch (KiCad schematic)
At the start: 9 parts, among them U201 AP63205WU, U202 TLV1117-33

Commit message: finished...
Parts:
- L201: LCSC C5331021 -> C2045343
Changed lines of the file:
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@@
 	(title_block
 		(title "Relay Control Board")
-		(date "2024-07-01")
-		(rev "PA")
+		(date "2024-07-09")
+		(rev "R1")
 		(company "UBC ThunderBikes")
 		(comment 1 "Peter Woolsey")
@@
 		(fill
 			(type none)
-		)
-	)
-	(text_box "I DIDN'T HAVE TIME TO RE-IMPLEMENT THE 24V-12V BUCK, THIS MEANS AN EXTERNAL BUCK WILL BE REQUIRED, BUT THE PUMP CAN STILL BE CONTROLLED WITH A SINGLE WIRE INTO THE BOARD."
-		(exclude_from_sim no)
-		(at 49.53 143.51 0)
-		(size 85.09 20.32)
-		(stroke
-			(width 0)
-			(type default)
-		)
-		(fill
-			(type color)
-			(color 194 0 0 1)
-		)
-		(effects
-			(font
-				(size 2 2)
-				(color 255 255 255 1)
-			)
-			(justify left top)
 		)
 	)
@@
 			)
 		)
-		(property "LCSC" "C5331021"
+		(property "LCSC" "C2045343"
 			(at 104.14 81.28 90)
 			(effects
