File: hv.kicad_sch (KiCad schematic)
At the start: 36 parts, among them Q701 IPD70R360P7S, U701 LM5168FDDAR, U702 AMC1311QDWVR, U703 TLV9001IDCK, U704 SN74LVC1G14DBV

Commit message: started working on it
Parts:
- removed C709: 2u2, Capacitor_SMD:C_0603_1608Metric, symbol Device:C_Small
- removed L701: 56u, Inductor_SMD:L_1210_3225Metric, symbol Device:L
- removed U701: LM5168FDDAR, Package_SO:TI_SO-PowerPAD-8, symbol 2024-05-06_02-50-10:LM5168FDDAR
- added D702, D703: DFLS1200-7, Diode_SMD_AKL:D_PowerDI-123, symbol PCM_Diode_Schottky_AKL:D_Schottky_Generic
- added L701: 560u, symbol Device:L_Small
- added U701: UCC28881DR, D0007A_N, symbol 2024-07-09_05-33-38:UCC28881DR
- C701: value 1u -> 220n; footprint Capacitor_SMD:C_1812_4532Metric_Pad1.57x3.40mm_HandSolder -> (none); LCSC C3037685 -> (none)
- C705: value 2n2 -> 10u; footprint Capacitor_SMD:C_0603_1608Metric -> (none); LCSC C107082 -> (none)
- C706: value 56p -> 100n; footprint Capacitor_SMD:C_0603_1608Metric -> (none); LCSC C1676 -> (none)
- C708: value 1n2 -> 100u; footprint Capacitor_SMD:C_0603_1608Metric -> (none); LCSC C107073 -> (none)
- R701: value 22k1 -> 10; footprint Resistor_SMD:R_0603_1608Metric -> (none); LCSC C25961 -> (none)
- R709: value 340k -> 44k2; footprint Resistor_SMD:R_0603_1608Metric -> (none); LCSC C2933203 -> (none)
- R712: value 316k -> 10k; footprint Resistor_SMD:R_0603_1608Metric -> (none); LCSC C2998125 -> (none)
- R713: value 101k -> 11k8; footprint Resistor_SMD:R_0603_1608Metric -> Resistor_SMD_AKL:R_0402_1005Metric; LCSC C862847 -> C481934
Connections:
- net HS+5V: now also R713.1, D702.2 (A), L701.2; no longer R712.1
- net HSGND: now also C705.1, C708.1, D703.2 (A); no longer C701.2, R701.2
- net V_MTRCTRL: now also R701.2; no longer C701.1
- net at C705.2: now also R701.1, U701.5 (HVIN), U701.8 (DRAIN); no longer R709.1
- new net: C701.1, C706.1, D703.1 (K), L701.1, R712.2, U701.1 (GND), U701.2 (GND)
- new net: C706.2, U701.4 (VDD)
- new net: R709.1, R712.1, U701.3 (FB)
- new net: C701.2, D702.1 (K), R709.2
Other:
- moved on the sheet: C707, C710, D701, R710, R711, R714, R715, R718, U703

Commit message: finished...
Parts:
- removed C705: 10u, symbol Device:C_Small
- added C705: 10u, Capacitor_THT:CP_Radial_D10.0mm_P5.00mm, symbol Device:C_Polarized_Small_US
- C701: footprint (none) -> Capacitor_SMD:C_0603_1608Metric; LCSC (none) -> C21120
- C706: footprint (none) -> Capacitor_SMD:C_0603_1608Metric; LCSC (none) -> C1591
- C708: footprint (none) -> Capacitor_SMD:C_1206_3216Metric; LCSC (none) -> C15008
- L701: value 560u -> 680u; footprint (none) -> Inductor_SMD:L_12x12mm_H8mm; LCSC (none) -> C2455611
- R701: footprint (none) -> Resistor_SMD:R_0603_1608Metric; LCSC (none) -> C22859
- R709: footprint (none) -> Resistor_SMD:R_0603_1608Metric; LCSC (none) -> C23056
- R712: footprint (none) -> Resistor_SMD:R_0603_1608Metric; LCSC (none) -> C25804
- U701: footprint D0007A_N -> footprints:D0007A_N
Connections:
- net HSGND: now also C705.2
- net at R701.1, U701.5 (HVIN), U701.8 (DRAIN): now also C705.1
Other:
- note added: "DISCHARGE CIRCUIT"
- note added: "DOUBLE ENDED TO SINGLE ENDED AMP"
- note added: "HV DC-DC CONVERTER"
- moved on the sheet: C701, C702, C703, C704, C706, C708, D701, D702, D703, L701, OC701, Q701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

Commit message: switched to an isolated dcdc transformer from LS 5V
Parts:
- removed C705: 10u, Capacitor_THT:CP_Radial_D10.0mm_P5.00mm, symbol Device:C_Polarized_Small_US
- removed C706: 100n, Capacitor_SMD:C_0603_1608Metric, symbol Device:C_Small
- removed C708: 100u, Capacitor_SMD:C_1206_3216Metric, symbol Device:C_Small
- removed D702, D703: DFLS1200-7, Diode_SMD_AKL:D_PowerDI-123, symbol PCM_Diode_Schottky_AKL:D_Schottky_Generic
- removed L701: 680u, Inductor_SMD:L_12x12mm_H8mm, symbol Device:L_Small
- removed R701: 10, Resistor_SMD:R_0603_1608Metric, symbol Device:R_Small
- removed R709: 44k2, Resistor_SMD:R_0603_1608Metric, symbol Device:R_Small
- removed R712: 10k, Resistor_SMD:R_0603_1608Metric, symbol Device:R_Small
- removed R713: 11k8, Resistor_SMD_AKL:R_0402_1005Metric, symbol Device:R_Small
- removed U701: UCC28881DR, footprints:D0007A_N, symbol 2024-07-09_05-33-38:UCC28881DR
- added C702: 4u7, Capacitor_SMD:C_0603_1608Metric, symbol Device:C_Small
- added U701: TMA-0505S, Converter_DCDC:Converter_DCDC_TRACO_TMA-05xxS_12xxS_Single_THT, symbol Converter_DCDC:TMA-0505S
- C701: value 220n -> 4u7; LCSC C21120 -> C108342
- renumbered C702 to C705, C707 to C706, C710 to C707
Connections:
- net GND: now also C701.2, C702.2, U701.2 (-Vin)
- net HS+5V: now also U701.6 (+Vout)
- net HSGND: now also U701.4 (-Vout)
- net +5V: now reaches C701.1
- net +5V: now also C702.1, U701.1 (+Vin)
- no-connect marks 1 -> 0
Other:
- note removed: "HV DC-DC CONVERTER"
- moved on the sheet: D701, R718
